File: pcb/senzory.kicad_sch (KiCad schematic)
At the start: 21 parts, among them J3 Ultrasonic eyes, Q1 S8050, Q2 AO3401A, U4 CD4052B, U5 QRE1113GR, U6 QRE1113GR, U7 QRE1113GR

Commit message: pridano par veci
Parts:
- removed Q1: S8050, Package_TO_SOT_SMD:SOT-23, symbol Transistor_BJT:S8050
- removed R7: 10k, Resistor_SMD:R_0603_1608Metric, symbol Device:R
- added JP1: Jumper_3_Bridged12, Connector_PinHeader_2.54mm:PinHeader_1x03_P2.54mm_Vertical, symbol Jumper:Jumper_3_Bridged12
Connections:
- net IR_0 is gone; now on net LED_PWR: R1.1
- net +3V3: now also Q2.2 (S), R8.2, JP1.1 (A)
- net +BATT: now also JP1.3 (B); no longer Q2.2 (S), R8.2
- net IR_ENABLE: now also Q2.1 (G), R8.1
- net DRV_A renamed LED_PWR
