File: pcb/senzory.kicad_sch (KiCad schematic)
At the start: 45 parts, among them J3 Ultrasonic eyes, Q2 AO3401A, U10 QRE1113GR, U11 QRE1113GR, U12 QRE1113GR, U4 CD4052B, U5 QRE1113GR, U6 QRE1113GR, U7 QRE1113GR, U8 QRE1113GR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

Commit message: schéma začátek pcb1
Parts:
- renumbered J3 to J4
Changed lines of the file:
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@@
 		(dnp no)
 		(fields_autoplaced yes)
-		(property "Reference" "J3"
+		(property "Reference" "J4"
 			(at 266.7 147.3199 0)
 			(effects
@@
 			(project "pcb"
 				(path "/fa68a0a1-2442-44ac-8421-6b9a18e1b14b/6193b7f2-5a02-49b0-b221-cbfe652a7ac1"
-					(reference "J3")
+					(reference "J4")
 					(unit 1)
 				)
