File: pcb/pcb.kicad_sch (KiCad schematic)
At the start: 54 parts, among them J1 Conn_01x20, J2 Conn_01x20, J3 Battery, J4 Ultrasonic eyes, M1 Motor_L, M2 Motor_R, Q1 AO3401A, U1 QRE1113GR, U10 DRV8220SDG, U2 QRE1113GR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

Commit message: Zapojení senzorů
Connections:
- net SENSOR_2: now also J2.15 (Pin_15)
- net SENSOR_3: now also J2.14 (Pin_14)
- net SENSOR_5: now also J1.15 (Pin_15)
- net SENSOR_6: now also J1.16 (Pin_16)
- net SENSOR_7: now also J1.17 (Pin_17)
Changed lines of the file:
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@@
+	(wire
+		(pts
+			(xy 135.89 57.15) (xy 148.59 57.15)
+		)
+		(stroke
+			(width 0)
+			(type default)
+		)
+	)
 	(wire
 		(pts
@@
 	(wire
 		(pts
+			(xy 97.79 62.23) (xy 110.49 62.23)
+		)
+		(stroke
+			(width 0)
+			(type default)
+		)
+	)
+	(wire
+		(pts
 			(xy 97.79 57.15) (xy 110.49 57.15)
 		)
@@
 	(wire
 		(pts
+			(xy 135.89 59.69) (xy 148.59 59.69)
+		)
+		(stroke
+			(width 0)
+			(type default)
+		)
+	)
+	(wire
+		(pts
 			(xy 15.24 177.8) (xy 26.67 177.8)
 		)
@@
 	(wire
 		(pts
+			(xy 97.79 64.77) (xy 110.49 64.77)
+		)
+		(stroke
+			(width 0)
+			(type default)
+		)
+	)
+	(wire
+		(pts
 			(xy 198.12 36.83) (xy 203.2 36.83)
 		)
@@
 		(pts
 			(xy 203.2 44.45) (xy 209.55 44.45)
+		)
+		(stroke
+			(width 0)
+			(type default)
+		)
+	)
+	(wire
+		(pts
+			(xy 97.79 59.69) (xy 110.49 59.69)
 		)
 		(stroke
@@
 		)
 	)
+	(label "SENSOR_6"
+		(at 97.79 62.23 0)
+		(effects
+			(font
+				(size 1.27 1.27)
+			)
+			(justify left bottom)
+		)
+	)
 	(label "MODE"
 		(at 100.33 44.45 0)
@@
 		)
 	)
+	(label "SENSOR_5"
+		(at 97.79 59.69 0)
+		(effects
+			(font
+				(size 1.27 1.27)
+			)
+			(justify left bottom)
+		)
+	)
 	(label "~{SLEEP}"
 		(at 100.33 46.99 0)
@@
 		)
 	)
+	(label "SENSOR_7"
+		(at 97.79 64.77 0)
+		(effects
+			(font
+				(size 1.27 1.27)
+			)
+			(justify left bottom)
+		)
+	)
 	(label "SENSOR_2"
 		(at 85.09 104.14 180)
@@
 		)
 	)
+	(label "SENSOR_3"
+		(at 148.59 57.15 180)
+		(effects
+			(font
+				(size 1.27 1.27)
+			)
+			(justify right bottom)
+		)
+	)
 	(label "~{SLEEP}"
 		(at 170.18 29.21 0)
@@
 		(effects
 			(font
+				(size 1.27 1.27)
+			)
+			(justify right bottom)
+		)
+	)
+	(label "SENSOR_2"
+		(at 148.59 59.69 180)
+		(effects
+			(font
