File: pcb/pcb.kicad_pcb (KiCad board)
At the start: 2 copper layers, 57 parts, among them J1 Battery, J2 R_GPIO, J3 L_GPIO, J4 Ultrasonic eyes, M1 Motor_L, M2 Motor_R, Q2 AO3401A, U1 DRV8220SDG, U10 QRE1113GR, U11 QRE1113GR, U12 QRE1113GR, U2 DRV8220SDG, U4 CD4052B, U5 QRE1113GR, U6 QRE1113GR, U7 QRE1113GR, U8 QRE1113GR, U9 QRE1113GR

Commit message: pcb
Parts:
- added BATT1: 18650, easyeda2kicad:BATTERY-SMD_18650-1S-L77.1-W20.7-1, F.Cu at (254.0, 90.5)
- added Q12: FS8205A_C2830320, easyeda2kicad:SOT-23-6_L2.9-W1.6-P0.95-LS2.8-BR, F.Cu at (95.8, 151.0)
- added U3: DW01A_C18164398, easyeda2kicad:SOT-23-6_L2.9-W1.6-P0.95-LS2.8-BR, F.Cu at (113.7, 150.9)
- moved U4 18.3 mm to (145.0, 151.5)
- moved R17 4.61 mm to (175.6, 98.5)
- moved R16 4.57 mm to (175.4, 94.0)
- moved R11 4.50 mm to (168.5, 98.5)
- moved R7 4.50 mm to (168.5, 94.0)
- moved U2 0.71 mm to (68.5, 81.2)

Commit message: Úpravy pro zjednodušení
Parts:
- removed BATT1: 18650, easyeda2kicad:BATTERY-SMD_18650-1S-L77.1-W20.7-1
- removed C17: 100n, Capacitor_SMD:C_0603_1608Metric_Pad1.08x0.95mm_HandSolder
- removed Q12: FS8205A_C2830320, easyeda2kicad:SOT-23-6_L2.9-W1.6-P0.95-LS2.8-BR
- removed Q2: AO3401A, Package_TO_SOT_SMD:SOT-23
- removed R21: 2,2k, Resistor_SMD:R_0603_1608Metric
- removed R22, R23: 10k, Resistor_SMD:R_0603_1608Metric
- removed U11, U12: QRE1113GR, OptoDevice:OnSemi_CASE100CY
- added D1: 1N4007, Diode_THT:D_A-405_P10.16mm_Horizontal, F.Cu at (223.5, 109.9)
- added Q1: AO3401A, Package_TO_SOT_SMD:SOT-23, F.Cu at (237.8, 127.0)
- added R18: 120, Resistor_SMD:R_0603_1608Metric_Pad0.98x0.95mm_HandSolder, F.Cu at (237.1, 99.0)
- C10, C14, C16, C6, C8: value 10u -> 100n
- C11, C13, C15, C7: value 100n -> 10u
- C5: value 100nF -> 10u; footprint Capacitor_SMD:C_0603_1608Metric -> Capacitor_SMD:C_0603_1608Metric_Pad1.08x0.95mm_HandSolder
- J1: footprint Connector_JST:JST_PH_S2B-PH-K_1x02_P2.00mm_Horizontal -> easyeda2kicad:BATTERY-SMD_18650-1S-L77.1-W20.7-1; moved to B.Cu
- J2: value R_GPIO -> Conn_01x20; footprint Connector_PinHeader_2.54mm:PinHeader_1x15_P2.54mm_Vertical -> Connector_PinSocket_2.54mm:PinSocket_1x20_P2.54mm_Vertical
- J3: value L_GPIO -> Conn_01x20; footprint Connector_PinHeader_2.54mm:PinHeader_1x15_P2.54mm_Vertical -> Connector_PinSocket_2.54mm:PinSocket_1x20_P2.54mm_Vertical
- R1, R16, R3, R7: value 120 -> 10k
- R13, R6: value 10k -> 120
- R15: footprint Resistor_SMD:R_0603_1608Metric_Pad0.98x0.95mm_HandSolder -> Resistor_SMD:R_0603_1608Metric
- R19: value 330 -> 120; footprint Resistor_SMD:R_0603_1608Metric -> Resistor_SMD:R_0603_1608Metric_Pad0.98x0.95mm_HandSolder
- R8: footprint Resistor_SMD:R_0603_1608Metric -> Resistor_SMD:R_0603_1608Metric_Pad0.98x0.95mm_HandSolder
- U1, U2: value DRV8220SDG -> QRE1113GR; footprint Package_SON:WSON-8-1EP_2x2mm_P0.5mm_EP0.9x1.6mm -> OptoDevice:OnSemi_CASE100CY
- U3: value DW01A_C18164398 -> QRE1113GR; footprint easyeda2kicad:SOT-23-6_L2.9-W1.6-P0.95-LS2.8-BR -> OptoDevice:OnSemi_CASE100CY
- U4: value CD4052B -> QRE1113GR; footprint Package_SO:SOIC-16W_5.3x10.2mm_P1.27mm -> OptoDevice:OnSemi_CASE100CY
- U5, U6: value QRE1113GR -> DRV8220SDG; footprint OptoDevice:OnSemi_CASE100CY -> Package_SON:WSON-8-1EP_2x2mm_P0.5mm_EP0.9x1.6mm
- moved M1 190.3 mm to (242.7, 88.5)
- moved M2 178.5 mm to (242.7, 96.3)
- moved U1 162.9 mm to (217.0, 79.7)
- moved U2 160.6 mm to (229.1, 81.6)
- moved U3 138.9 mm to (234.0, 81.6)
- moved R19 125.9 mm to (237.1, 101.5)
- moved U4 117.0 mm to (238.8, 81.6)
- moved U5 115.2 mm to (237.6, 119.3)
- moved C5 113.2 mm to (224.0, 96.5)
- moved U6 108.1 mm to (237.6, 123.0)
- moved J1 106.9 mm to (90.0, 100.0), turned to 180 degrees
- moved U7 101.7 mm to (243.6, 81.6)
- moved R1 101.5 mm to (228.4, 104.0)
- moved R2 101.2 mm to (228.4, 106.5)
- moved C2 98.6 mm to (224.0, 88.9)
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Connections:
- net /GP9 renamed VBUS
- C1 pad 1: Net-(U5-A) -> Net-(U1-A)
- C10 pad 1: Net-(U10-A) -> /SENSOR_2
- C11 pad 1: /Senzory/SENSOR_4 -> Net-(U8-A)
- C12 pad 1: /Senzory/SENSOR_5 -> /SENSOR_6
- C13 pad 1: /Senzory/SENSOR_6 -> Net-(U9-A)
- C14 pad 1: Net-(U11-A) -> /SENSOR_3
- C15 pad 1: /Senzory/SENSOR_3 -> Net-(U10-A)
- C16 pad 1: Net-(U12-A) -> /SENSOR_7
- C2 pad 1: /Senzory/SENSOR_0 -> /SENSOR_0
- C3 pad 1: Net-(U6-A) -> Net-(U2-A)
- C4 pad 1: /Senzory/SENSOR_1 -> /SENSOR_4
- C5 pad 1: /BVDD -> Net-(U3-A)
- C5 pad 2: -BATT -> GND
- C6 pad 1: Net-(U7-A) -> /SENSOR_1
- C7 pad 1: /Senzory/SENSOR_2 -> Net-(U4-A)
- C8 pad 1: Net-(U8-A) -> /SENSOR_5
- C9 pad 1: Net-(U9-A) -> Net-(U7-A)
- J1 pad 1: unconnected-(J1-Pin_1-Pad1) -> GND
- J1 pad 2: unconnected-(J1-Pin_2-Pad2) -> Net-(D1-A)
- J2 pad 1: /GP0 -> unconnected-(J2-Pin_1-Pad1)
- J2 pad 10: /GP7 -> /~{SLEEP}
- J2 pad 11: /GP8 -> /TRIG
- J2 pad 12: /RXD -> /ECHO
- J2 pad 13: /TXD -> GND
- J2 pad 14: GND -> /SENSOR_4
- J2 pad 15: +3V3 -> unconnected-(J2-Pin_15-Pad15)
- J2 pad 2: /GP1 -> unconnected-(J2-Pin_2-Pad2)
- J2 pad 3: /GP2 -> GND
- J2 pad 4: /GP3 -> unconnected-(J2-Pin_4-Pad4)
- J2 pad 5: /GP4 -> unconnected-(J2-Pin_5-Pad5)
- J2 pad 6: /GP5 -> unconnected-(J2-Pin_6-Pad6)
- J2 pad 7: GND -> unconnected-(J2-Pin_7-Pad7)
- J2 pad 8: +3V3 -> GND
- J2 pad 9: /GP6 -> /MODE
- J3 pad 10: GND -> /VBAT/2
- J3 pad 11: +3V3 -> unconnected-(J3-Pin_11-Pad11)
- J3 pad 12: /EN -> /~{IR_ENABLE}
- J3 pad 13: /RST -> GND
- J3 pad 14: GND -> unconnected-(J3-Pin_14-Pad14)
- J3 pad 15: VIN -> unconnected-(J3-Pin_15-Pad15)
- J3 pad 2: GND -> +BATT
- J3 pad 3: VUSB -> GND
- J3 pad 4: /GP10 -> unconnected-(J3-Pin_4-Pad4)
- J3 pad 5: /GP11 -> +3V3
- J3 pad 6: /GP12 -> unconnected-(J3-Pin_6-Pad6)
- J3 pad 7: /GP13 -> unconnected-(J3-Pin_7-Pad7)
- J3 pad 8: /GP14 -> GND
- J3 pad 9: /GP15 -> unconnected-(J3-Pin_9-Pad9)
- J4 pad 1: +3V3 -> Net-(J4-Pin_1)
- J4 pad 2: /GP4 -> /TRIG
- J4 pad 3: /GP3 -> /ECHO
- JP1 pad 2: unconnected-(JP1-C-Pad2) -> Net-(J4-Pin_1)
- R1 pad 1: /Senzory/LED_PWR -> Net-(D1-A)
- R1 pad 2: Net-(U5-A) -> /VBAT/2
- R10 pad 1: /Senzory/LED_PWR -> /LED_PWR
- R10 pad 2: Net-(U10-A) -> Net-(U4-A)
- R11 pad 1: /Senzory/SENSOR_4 -> /SENSOR_2
- R12 pad 1: /Senzory/SENSOR_5 -> /SENSOR_6
- R13 pad 1: /Senzory/SENSOR_6 -> /LED_PWR
- R13 pad 2: +3V3 -> Net-(U7-A)
- R14 pad 1: /Senzory/LED_PWR -> /LED_PWR
- R14 pad 2: Net-(U11-A) -> Net-(U8-A)
- R15 pad 1: /Senzory/SENSOR_3 -> /~{IR_ENABLE}
- R16 pad 1: /Senzory/LED_PWR -> /SENSOR_3
- R16 pad 2: Net-(U12-A) -> +3V3
- R17 pad 1: /Senzory/SENSOR_7 -> /SENSOR_7
- R19 pad 1: /BVDD -> /LED_PWR
- R19 pad 2: +BATT -> Net-(U10-A)
- R2 pad 1: /Senzory/SENSOR_0 -> /VBAT/2
- R2 pad 2: +3V3 -> GND
- R3 pad 1: /Senzory/LED_PWR -> /SENSOR_0
- R3 pad 2: Net-(U6-A) -> +3V3
- R4 pad 1: /Senzory/SENSOR_1 -> /SENSOR_4
- R5 pad 1: /Senzory/LED_PWR -> /LED_PWR
- R5 pad 2: Net-(U7-A) -> Net-(U1-A)
- R6 pad 1: /Senzory/SENSOR_2 -> /LED_PWR
- R6 pad 2: +3V3 -> Net-(U2-A)
- R7 pad 1: /Senzory/LED_PWR -> /SENSOR_1
- R7 pad 2: Net-(U8-A) -> +3V3
- R8 pad 1: /GP8 -> /SENSOR_5
- R9 pad 1: /Senzory/LED_PWR -> /LED_PWR
- R9 pad 2: Net-(U9-A) -> Net-(U3-A)
- U1 pad 1: +BATT -> Net-(U1-A)
- U1 pad 2: Net-(M1-+) -> GND
- U1 pad 3: Net-(M1--) -> /SENSOR_0
- U10 pad 3: /Senzory/SENSOR_6 -> /SENSOR_7
- U2 pad 1: +BATT -> Net-(U2-A)
- U2 pad 2: Net-(M2-+) -> GND
- U2 pad 3: Net-(M2--) -> /SENSOR_4
- U3 pad 1: Net-(Q12-G1) -> Net-(U3-A)
- U3 pad 2: Net-(U3-VM) -> GND
- U3 pad 3: Net-(Q12-G2) -> /SENSOR_1
- U3 pad 4: unconnected-(U3-NC-Pad4) -> GND
- U4 pad 1: /Senzory/SENSOR_4 -> Net-(U4-A)
- U4 pad 2: /Senzory/SENSOR_6 -> GND
- U4 pad 3: /GP6 -> /SENSOR_5
- U4 pad 4: /Senzory/SENSOR_7 -> GND
- U5 pad 1: Net-(U5-A) -> +BATT
- U5 pad 2: GND -> Net-(M1-+)
- U5 pad 3: /Senzory/SENSOR_0 -> Net-(M1--)
- U6 pad 1: Net-(U6-A) -> +BATT
- U6 pad 2: GND -> Net-(M2-+)
- U6 pad 3: /Senzory/SENSOR_1 -> Net-(M2--)
- U7 pad 3: /Senzory/SENSOR_2 -> /SENSOR_2
- U8 pad 3: /Senzory/SENSOR_4 -> /SENSOR_6
- U9 pad 3: /Senzory/SENSOR_5 -> /SENSOR_3
Routing:
- added copper zone on B.Cu, net GND
- added copper zone on F.Cu, net GND
Other:
- board outline added: 80 x 144.2 mm

Commit message: Úklid schématu
Parts:
- C10, C12, C2, C4: value 100n -> 10u
- C13, C15, C5, C7: value 10u -> 100n
- J1: value Battery -> Conn_01x20; footprint easyeda2kicad:BATTERY-SMD_18650-1S-L77.1-W20.7-1 -> Connector_PinSocket_2.54mm:PinSocket_1x20_P2.54mm_Vertical
- J3: value Conn_01x20 -> Battery; footprint Connector_PinSocket_2.54mm:PinSocket_1x20_P2.54mm_Vertical -> easyeda2kicad:BATTERY-SMD_18650-1S-L77.1-W20.7-1
- R1, R11, R12, R2, R3, R4: value 10k -> 120
- R13, R14, R18, R19, R5, R6: value 120 -> 10k
- R15: footprint Resistor_SMD:R_0603_1608Metric -> Resistor_SMD:R_0603_1608Metric_Pad0.98x0.95mm_HandSolder
- R17: footprint Resistor_SMD:R_0603_1608Metric_Pad0.98x0.95mm_HandSolder -> Resistor_SMD:R_0603_1608Metric
- U10, U9: value QRE1113GR -> DRV8220SDG; footprint OptoDevice:OnSemi_CASE100CY -> Package_SON:WSON-8-1EP_2x2mm_P0.5mm_EP0.9x1.6mm
- U5, U6: value DRV8220SDG -> QRE1113GR; footprint Package_SON:WSON-8-1EP_2x2mm_P0.5mm_EP0.9x1.6mm -> OptoDevice:OnSemi_CASE100CY
- moved J3 46.8 mm to (90.0, 100.0), turned to 0 degrees
- moved J1 46.6 mm to (98.9, 145.7), turned to 0 degrees
- moved J2 19.0 mm to (81.1, 145.7)
Connections:
- C10 pad 1: /SENSOR_2 -> Net-(U6-A)
- C11 pad 1: Net-(U8-A) -> Net-(U7-A)
- C12 pad 1: /SENSOR_6 -> Net-(U8-A)
- C13 pad 1: Net-(U9-A) -> /SENSOR_4
- C14 pad 1: /SENSOR_3 -> /SENSOR_5
- C15 pad 1: Net-(U10-A) -> /SENSOR_6
- C2 pad 1: /SENSOR_0 -> Net-(U2-A)
- C3 pad 1: Net-(U2-A) -> Net-(U3-A)
- C4 pad 1: /SENSOR_4 -> Net-(U4-A)
- C5 pad 1: Net-(U3-A) -> /SENSOR_0
- C7 pad 1: Net-(U4-A) -> /SENSOR_2
- C8 pad 1: /SENSOR_5 -> /SENSOR_3
- C9 pad 1: Net-(U7-A) -> Net-(U5-A)
- J1 pad 1: GND -> unconnected-(J1-Pin_1-Pad1)
- J1 pad 2: Net-(D1-A) -> unconnected-(J1-Pin_2-Pad2)
- J2 pad 1: unconnected-(J2-Pin_1-Pad1) -> VBUS
- J2 pad 10: /~{SLEEP} -> /VBAT/2
- J2 pad 11: /TRIG -> unconnected-(J2-Pin_11-Pad11)
- J2 pad 12: /ECHO -> /~{IR_ENABLE}
- J2 pad 14: /SENSOR_4 -> unconnected-(J2-Pin_14-Pad14)
- J2 pad 16: unconnected-(J2-Pin_16-Pad16) -> /SENSOR_1
- J2 pad 17: unconnected-(J2-Pin_17-Pad17) -> /SENSOR_0
- J2 pad 19: /MOT_L_A -> /MOT_R_A
- J2 pad 2: unconnected-(J2-Pin_2-Pad2) -> +BATT
- J2 pad 20: /MOT_L_B -> /MOT_R_B
- J2 pad 5: unconnected-(J2-Pin_5-Pad5) -> +3V3
- J2 pad 9: /MODE -> unconnected-(J2-Pin_9-Pad9)
- J3 pad 1: VBUS -> GND
- J3 pad 2: +BATT -> Net-(D1-A)
- R1 pad 1: Net-(D1-A) -> /LED_PWR
- R1 pad 2: /VBAT/2 -> Net-(U1-A)
- R10 pad 2: Net-(U4-A) -> Net-(U6-A)
- R11 pad 1: /SENSOR_2 -> /LED_PWR
- R11 pad 2: +3V3 -> Net-(U7-A)
- R12 pad 1: /SENSOR_6 -> /LED_PWR
- R12 pad 2: +3V3 -> Net-(U8-A)
- R13 pad 1: /LED_PWR -> /SENSOR_4
- R13 pad 2: Net-(U7-A) -> +3V3
- R14 pad 1: /LED_PWR -> /SENSOR_5
- R14 pad 2: Net-(U8-A) -> +3V3
- R15 pad 1: /~{IR_ENABLE} -> /SENSOR_6
- R16 pad 1: /SENSOR_3 -> /SENSOR_7
- R17 pad 1: /SENSOR_7 -> /~{IR_ENABLE}
- R18 pad 1: /LED_PWR -> Net-(D1-A)
- R18 pad 2: Net-(U9-A) -> /VBAT/2
- R19 pad 1: /LED_PWR -> /VBAT/2
- R19 pad 2: Net-(U10-A) -> GND
- R2 pad 1: /VBAT/2 -> /LED_PWR
- R2 pad 2: GND -> Net-(U2-A)
- R3 pad 1: /SENSOR_0 -> /LED_PWR
- R3 pad 2: +3V3 -> Net-(U3-A)
- R4 pad 1: /SENSOR_4 -> /LED_PWR
- R4 pad 2: +3V3 -> Net-(U4-A)
- R5 pad 1: /LED_PWR -> /SENSOR_0
- R5 pad 2: Net-(U1-A) -> +3V3
- R6 pad 1: /LED_PWR -> /SENSOR_1
- R6 pad 2: Net-(U2-A) -> +3V3
- R7 pad 1: /SENSOR_1 -> /SENSOR_2
- R8 pad 1: /SENSOR_5 -> /SENSOR_3
- R9 pad 2: Net-(U3-A) -> Net-(U5-A)
- U10 pad 1: Net-(U10-A) -> +BATT
- U10 pad 2: GND -> Net-(M2-+)
- U10 pad 3: /SENSOR_7 -> Net-(M2--)
- U2 pad 3: /SENSOR_4 -> /SENSOR_1
- U3 pad 3: /SENSOR_1 -> /SENSOR_2
- U4 pad 3: /SENSOR_5 -> /SENSOR_3
- U5 pad 1: +BATT -> Net-(U5-A)
- U5 pad 2: Net-(M1-+) -> GND
- U5 pad 3: Net-(M1--) -> /SENSOR_4
- U6 pad 1: +BATT -> Net-(U6-A)
- U6 pad 2: Net-(M2-+) -> GND
- U6 pad 3: Net-(M2--) -> /SENSOR_5
- U7 pad 3: /SENSOR_2 -> /SENSOR_6
- U8 pad 3: /SENSOR_6 -> /SENSOR_7
- U9 pad 1: Net-(U9-A) -> +BATT
- U9 pad 2: GND -> Net-(M1-+)
- U9 pad 3: /SENSOR_3 -> Net-(M1--)

Commit message: Zapojení senzorů
Parts:
- C1, C10, C11, C12, C13, C14, C15, C16, C2, C3, C4, C5, C6, C7, C8, C9, J3, R1, R10, R11, R12, R13, R14, R15, R16, R2, R3, R4, R5, R6, R7, R8, R9, U1, U2, U3, U4, U5, U6, U7, U8: moved to B.Cu
- J1: moved to F.Cu
- moved U10 187.6 mm to (72.0, 57.5)
- moved R5 185.3 mm to (52.1, 50.3), turned to 90 degrees
- moved M2 183.2 mm to (63.8, 57.5)
- moved R1 178.9 mm to (57.7, 50.3), turned to -90 degrees
- moved R6 177.4 mm to (62.2, 45.1), turned to 90 degrees
- moved C5 177.2 mm to (52.1, 53.8), turned to -90 degrees
- moved R2 171.9 mm to (67.9, 45.1), turned to -90 degrees
- moved R7 169.6 mm to (72.2, 41.9), turned to 90 degrees
- moved C6 169.5 mm to (62.2, 48.6), turned to -90 degrees
- moved C1 169.5 mm to (57.7, 53.8), turned to -90 degrees
- moved U2 167.7 mm to (65.0, 46.9), turned to 180 degrees
- moved U1 164.4 mm to (54.9, 52.1), turned to 180 degrees
- moved U3 163.4 mm to (75.0, 43.7), turned to 180 degrees
- moved U5 162.1 mm to (95.0, 42.1), turned to 180 degrees
- moved C7 161.9 mm to (72.2, 45.4), turned to -90 degrees
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Routing:
- net /LED_PWR: track 0.00 -> 23.1 mm
- net Net-(U5-A): track 0.00 -> 4.17 mm
- net Net-(U4-A): track 0.00 -> 4.17 mm
- net /SENSOR_3: track 0.00 -> 4.15 mm
- net Net-(U2-A): track 0.00 -> 4.15 mm
- net /SENSOR_4: track 0.00 -> 4.15 mm
- net Net-(U6-A): track 0.00 -> 4.14 mm
- net /SENSOR_1: track 0.00 -> 4.14 mm
- net Net-(U7-A): track 0.00 -> 4.14 mm
- net /SENSOR_6: track 0.00 -> 4.13 mm
- net /SENSOR_2: track 0.00 -> 4.13 mm
- net /SENSOR_0: track 0.00 -> 4.13 mm
- net /SENSOR_5: track 0.00 -> 4.12 mm
- net Net-(U1-A): track 0.00 -> 4.11 mm
- net Net-(U8-A): track 0.00 -> 4.11 mm
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Other:
- board size 80 x 144.2 mm -> 80 x 129.2 mm

Commit message: Dodělané pcb
Parts:
- R18, R19: moved to B.Cu
- moved R18 79.3 mm to (78.1, 67.0), turned to 180 degrees
- moved R19 79.3 mm to (78.1, 69.5), turned to 180 degrees
- moved Q1 69.8 mm to (102.8, 56.0)
- moved D1 62.2 mm to (81.9, 75.0)
- moved R17 60.8 mm to (97.9, 55.0), turned to 180 degrees
- turned U9 to 180 degrees
Connections:
- J1 pad 15: unconnected-(J1-Pin_15-Pad15) -> /SENSOR_5
- J1 pad 16: unconnected-(J1-Pin_16-Pad16) -> /SENSOR_6
- J1 pad 17: unconnected-(J1-Pin_17-Pad17) -> /SENSOR_7
- J2 pad 14: unconnected-(J2-Pin_14-Pad14) -> /SENSOR_3
- J2 pad 15: unconnected-(J2-Pin_15-Pad15) -> /SENSOR_2
Routing:
- net GND: track 0.00 -> 312.3 mm, vias 0 -> 10
- net +BATT: track 0.00 -> 245.7 mm
- net +3V3: track 0.00 -> 216.7 mm
- net /MODE: track 0.00 -> 143.3 mm, vias 0 -> 2
- net /~{SLEEP}: track 0.00 -> 139.1 mm, vias 0 -> 3
- net /~{IR_ENABLE}: track 0.00 -> 131.8 mm
- net Net-(D1-A): track 0.00 -> 91.1 mm, vias 0 -> 1
- net /SENSOR_3: track 4.15 -> 76.3 mm
- net /SENSOR_2: track 4.13 -> 75.5 mm
- net /SENSOR_4: track 4.15 -> 71.3 mm
- net /SENSOR_1: track 4.14 -> 68.0 mm
- net /SENSOR_5: track 4.12 -> 66.4 mm
- net /TRIG: track 0.00 -> 61.4 mm
- net /SENSOR_6: track 4.13 -> 63.9 mm
- net /SENSOR_0: track 4.13 -> 63.7 mm
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
Commit message: pcb upravená cestička
Routing:
- net /SENSOR_2: track 75.5 -> 67.9 mm
- net /SENSOR_1: track 68.0 -> 65.5 mm
Changed lines of the file:
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@@
-	)
-	(segment
-		(start 85 96.08)
-		(end 81.11 99.97)
-		(width 0.4)
-		(layer "B.Cu")
-		(net 7)
-	)
-	(segment
-		(start 74.399 78.098884)
-		(end 74.502116 78.202)
-		(width 0.4)
-		(layer "B.Cu")
-		(net 7)
 	)
 	(segment
@@
 	)
 	(segment
-		(start 73.798 65.647942)
-		(end 73.798 76.502116)
+		(start 73.798 58.57039)
+		(end 64.1128 48.88519)
 		(width 0.4)
 		(layer "B.Cu")
@@
 	(segment
 		(start 85 88.699884)
-		(end 85 96.08)
+		(end 73.798 77.497884)
 		(width 0.4)
 		(layer "B.Cu")
@@
 	)
 	(segment
+		(start 73.798 77.497884)
+		(end 73.798 58.57039)
+		(width 0.4)
+		(layer "B.Cu")
+		(net 7)
+	)
+	(segment
 		(start 64.1128 48.88519)
 		(end 63.26809 48.88519)
@@
 	)
 	(segment
-		(start 74.502116 78.202)
-		(end 74.751058 78.450942)
-		(width 0.4)
-		(layer "B.Cu")
-		(net 7)
-	)
-	(segment
-		(start 73.798 76.502116)
-		(end 73.798 77)
-		(width 0.4)
-		(layer "B.Cu")
-		(net 7)
-	)
-	(segment
-		(start 74.150058 77.849942)
-		(end 74.399 78.098884)
-		(width 0.4)
-		(layer "B.Cu")
-		(net 7)
-	)
-	(segment
-		(start 74.751058 78.450942)
+		(start 81.11 99.97)
+		(end 85 96.08)
+		(width 0.4)
+		(layer "B.Cu")
+		(net 7)
+	)
+	(segment
+		(start 85 96.08)
 		(end 85 88.699884)
-		(width 0.4)
-		(layer "B.Cu")
-		(net 7)
-	)
-	(segment
-		(start 73.798 64.652174)
-		(end 73.798 65.150058)
-		(width 0.4)
-		(layer "B.Cu")
-		(net 7)
-	)
-	(segment
-		(start 74.150058 64.300116)
-		(end 73.798 64.652174)
-		(width 0.4)
-		(layer "B.Cu")
-		(net 7)
-	)
-	(segment
-		(start 73.798 77)
-		(end 73.798 77.497884)
-		(width 0.4)
-		(layer "B.Cu")
-		(net 7)
-	)
-	(segment
-		(start 76.838892 61.611282)
-		(end 74.502116 63.948058)
-		(width 0.4)
-		(layer "B.Cu")
-		(net 7)
-	)
-	(segment
-		(start 73.798 65.150058)
-		(end 73.798 65.647942)
-		(width 0.4)
-		(layer "B.Cu")
-		(net 7)
-	)
-	(segment
-		(start 73.798 77.497884)
-		(end 74.150058 77.849942)
-		(width 0.4)
-		(layer "B.Cu")
-		(net 7)
-	)
-	(segment
-		(start 64.1128 48.88519)
-		(end 76.838892 61.611282)
-		(width 0.4)
-		(layer "B.Cu")
-		(net 7)
-	)
-	(segment
-		(start 74.502116 63.948058)
-		(end 74.150058 64.300116)
 		(width 0.4)
 		(layer "B.Cu")
@@
 	)
 	(segment
-		(start 83.499 55.055551)
-		(end 83.499 55.801116)
-		(width 0.4)
-		(layer "B.Cu")
-		(net 12)
-	)
-	(segment
 		(start 73.298251 45.656551)
 		(end 72.1692 44.5275)
@@
 	)
 	(segment
-		(start 74.751058 64.549058)
-		(end 74.399 64.901116)
-		(width 0.4)
-		(layer "B.Cu")
-		(net 12)
-	)
-	(segment
-		(start 74.399 65.399)
-		(end 74.399 76.751058)
-		(width 0.4)
-		(layer "B.Cu")
-		(net 12)
-	)
-	(segment
-		(start 74.751058 77.601)
-		(end 75 77.849942)
-		(width 0.4)
-		(layer "B.Cu")
-		(net 12)
-	)
-	(segment
-		(start 74.399 76.751058)
-		(end 74.399 77.248942)
+		(start 74.399 77.248942)
+		(end 74.399 45.955551)
+		(width 0.4)
+		(layer "B.Cu")
+		(net 12)
+	)
+	(segment
+		(start 81.11 102.51)
+		(end 86 97.62)
 		(width 0.4)
 		(layer "B.Cu")
@@
 	(segment
 		(start 86 97.62)
-		(end 81.11 102.51)
-		(width 0.4)
-		(layer "B.Cu")
-		(net 12)
-	)
-	(segment
-		(start 74.399 64.901116)
-		(end 74.399 65.399)
+		(end 86 88.849942)
 		(width 0.4)
 		(layer "B.Cu")
@@
 	)
 	(segment
-		(start 75 77.849942)
-		(end 86 88.849942)
-		(width 0.4)
-		(layer "B.Cu")
-		(net 12)
-	)
-	(segment
 		(start 72.1692 42.7973)
 		(end 72.1692 44.5275)
@@
 	)
 	(segment
+		(start 74.399 45.955551)
+		(end 74.1 45.656551)
+		(width 0.4)
+		(layer "B.Cu")
+		(net 12)
+	)
+	(segment
 		(start 86 88.849942)
-		(end 86 97.62)
-		(width 0.4)
-		(layer "B.Cu")
-		(net 12)
-	)
-	(segment
-		(start 83.499 55.801116)
-		(end 74.751058 64.549058)
-		(width 0.4)
-		(layer "B.Cu")
-		(net 12)
-	)
-	(segment
-		(start 74.399 77.248942)
-		(end 74.751058 77.601)
-		(width 0.4)
-		(layer "B.Cu")
-		(net 12)
-	)
-	(segment
-		(start 74.1 45.656551)
-		(end 83.499 55.055551)
-		(width 0.4)
-		(layer "B.Cu")
+		(end 74.399 77.248942)
+		(width 0.4)
+		(layer "B.Cu")
